File: e_schemes/Reciever/Reciever/Reciever.kicad_pcb (KiCad board)
At the start: 2 copper layers, 36 parts, among them J1 Conn_01x03, J2 Conn_01x03, SW1 SW_Push, SW2 SW_Push, SW3 SW_Reload, U1 ESP32-WROOM-32E

Commit message: rx scheme1
Parts:
- added R16: 1М, Resistor_THT:R_Axial_DIN0204_L3.6mm_D1.6mm_P7.62mm_Horizontal, F.Cu at (209.8, 97.5)
- added U2: LM358, Package_DIP:DIP-8_W7.62mm_LongPads, F.Cu at (213.2, 92.1)
- added U3: LM393, Package_DIP:DIP-8_W7.62mm_LongPads, F.Cu at (199.2, 79.7)
- R3: value 2M -> 1М; footprint Resistor_THT:R_Axial_DIN0204_L3.6mm_D1.6mm_P7.62mm_Horizontal -> Resistor_THT:(DRILL)R_Axial_DIN0204_L3.6mm_D1.6mm_P7.62mm_Horizontal
- moved R6 137.4 mm to (209.8, 90.5), turned to 180 degrees
- moved J2 132.1 mm to (216.2, 54.8)
- moved R3 130.1 mm to (202.1, 95.0)
- moved R12 128.6 mm to (220.2, 72.0), turned to 180 degrees
- moved R11 127.4 mm to (220.4, 75.2), turned to 180 degrees
- moved R14 124.9 mm to (196.0, 80.1), turned to 90 degrees
- moved R10 124.5 mm to (218.3, 78.2), turned to 180 degrees
- moved R13 121.1 mm to (193.2, 87.6), turned to 90 degrees
- moved R7 120.0 mm to (191.3, 76.0), turned to 180 degrees
- moved C3 109.7 mm to (212.8, 58.5), turned to -90 degrees
- moved D1 109.6 mm to (219.6, 96.5), turned to 180 degrees
- moved C6 106.6 mm to (212.0, 97.8), turned to 90 degrees
- moved C4 102.5 mm to (207.5, 74.2)
- moved SW2 101.9 mm to (220.5, 65.5), turned to 180 degrees
- moved R15 101.8 mm to (196.5, 97.6), turned to 90 degrees
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Connections:
- R3 pad 1: Net-(D1-A) -> Net-(R16-Pad2)
Routing:
- net +3.3V: track 0.00 -> 94.5 mm
- net +5V: track 0.00 -> 49.5 mm
- net Net-(U3A-+): track 0.00 -> 32.6 mm
- net Net-(U1-IO19): track 0.00 -> 31.0 mm
- net Net-(U1-IO33): track 0.00 -> 25.3 mm
- net Net-(U1-IO32): track 0.00 -> 23.2 mm
- net Net-(U1-IO25): track 0.00 -> 21.4 mm
- net Net-(U1-IO18): track 0.00 -> 20.5 mm
- net Net-(U1-EN): track 0.00 -> 18.0 mm
- net Net-(U3A--): track 0.00 -> 17.9 mm
- net Net-(U1-IO34): track 0.00 -> 13.6 mm
- net Net-(J2-Pin_2): track 0.00 -> 11.3 mm
- net Net-(R13-Pad2): track 0.00 -> 10.9 mm
- net Net-(D1-A): track 0.00 -> 10.3 mm
- net Net-(D6-A): track 0.00 -> 9.89 mm
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- added copper zone on B.Cu, net GND
- added copper zone on F.Cu, net GND
Other:
- board outline added: 50 x 50 mm
