File: e_schemes/Reciever/Reciever/Reciever.kicad_sch (KiCad schematic)
At the start: 38 parts, among them J1 Conn_01x03, J2 Conn_01x03, SW1 SW_Push, SW2 SW_Push, SW3 SW_Reload, U1 ESP32-WROOM-32E, U2 LM358, U3 LM393

Commit message: rx scheme1
Parts:
- added R16: 1М, Resistor_THT:R_Axial_DIN0204_L3.6mm_D1.6mm_P7.62mm_Horizontal, symbol Device:R
- R3: value 2M -> 1М
- U2, U3: footprint (none) -> Package_DIP:DIP-8_W7.62mm_LongPads
Connections:
- net at C6.1, D1.2 (A), U2.2 (-): now also R16.1; no longer R3.1
- new net: R16.2, R3.1
Other:
- moved on the sheet: R3
Changed lines of the file:
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@@
 	(wire
 		(pts
-			(xy 208.28 82.55) (xy 208.28 105.41)
+			(xy 198.12 82.55) (xy 198.12 105.41)
 		)
 		(stroke
@@
 	(wire
 		(pts
+			(xy 209.55 46.99) (xy 209.55 95.25)
+		)
+		(stroke
+			(width 0)
+			(type default)
+		)
+	)
+	(wire
+		(pts
 			(xy 234.95 125.73) (xy 231.14 125.73)
 		)
@@
 	(wire
 		(pts
-			(xy 208.28 82.55) (xy 215.9 82.55)
+			(xy 198.12 82.55) (xy 215.9 82.55)
 		)
 		(stroke
@@
 	(wire
 		(pts
+			(xy 39.37 63.5) (xy 36.83 63.5)
+		)
+		(stroke
+			(width 0)
+			(type default)
+		)
+	)
+	(wire
+		(pts
 			(xy 231.14 46.99) (xy 231.14 38.1)
 		)
@@
 	(wire
 		(pts
-			(xy 50.8 63.5) (xy 58.42 63.5)
+			(xy 55.88 63.5) (xy 58.42 63.5)
 		)
 		(stroke
@@
 	(wire
 		(pts
-			(xy 43.18 63.5) (xy 36.83 63.5)
+			(xy 48.26 63.5) (xy 46.99 63.5)
 		)
 		(stroke
@@
 	(wire
 		(pts
-			(xy 209.55 46.99) (xy 209.55 95.25)
-		)
-		(stroke
-			(width 0)
-			(type default)
-		)
-	)
-	(wire
-		(pts
 			(xy 175.26 80.01) (xy 166.37 80.01)
 		)
@@
 	(wire
 		(pts
-			(xy 208.28 105.41) (xy 191.77 105.41)
+			(xy 198.12 105.41) (xy 191.77 105.41)
 		)
 		(stroke
@@
 			)
 		)
-		(property "Footprint" ""
+		(property "Footprint" "Package_DIP:DIP-8_W7.62mm_LongPads"
 			(at 48.26 48.26 0)
 			(effects
@@
 			)
 		)
-		(property "Footprint" ""
+		(property "Footprint" "Package_DIP:DIP-8_W7.62mm_LongPads"
 			(at 29.21 90.17 0)
 			(effects
@@
 			)
 		)
-		(property "Footprint" ""
+		(property "Footprint" "Package_DIP:DIP-8_W7.62mm_LongPads"
 			(at 26.67 118.11 0)
 			(effects
@@
 	(symbol
 		(lib_id "Device:R")
+		(at 43.18 63.5 90)
+		(unit 1)
+		(exclude_from_sim no)
+		(in_bom yes)
+		(on_board yes)
+		(dnp no)
+		(fields_autoplaced yes)
+		(property "Reference" "R16"
+			(at 43.18 57.15 90)
+			(effects
+				(font
+					(size 1.27 1.27)
+				)
+			)
+		)
+		(property "Value" "1М"
+			(at 43.18 59.69 90)
+			(effects
+				(font
+					(size 1.27 1.27)
+				)
+			)
+		)
+		(property "Footprint" "Resistor_THT:R_Axial_DIN0204_L3.6mm_D1.6mm_P7.62mm_Horizontal"
+			(at 43.18 65.278 90)
+			(effects
+				(font
+					(size 1.27 1.27)
+				)
+				(hide yes)
+			)
+		)
+		(property "Datasheet" "~"
+			(at 43.18 63.5 0)
+			(effects
+				(font
+					(size 1.27 1.27)
+				)
+				(hide yes)
+			)
+		)
+		(property "Description" "Resistor"
+			(at 43.18 63.5 0)
+			(effects
+				(font
+					(size 1.27 1.27)
+				)
+				(hide yes)
+			)
+		)
+		(pin "2"
+		)
+		(pin "1"
+		)
+		(instances
+			(project "Reciever"
+				(path "/340a7a4e-546f-4e6e-b22c-e44e009cc8c7"
+					(reference "R16")
+					(unit 1)
+				)
+			)
+		)
+	)
+	(symbol
+		(lib_id "Device:R")
 		(at 88.9 63.5 270)
 		(unit 1)
@@
 			)
 		)
-		(property "Footprint" ""
+		(property "Footprint" "Package_DIP:DIP-8_W7.62mm_LongPads"
 			(at 90.17 92.71 0)
 			(effects
@@
 			)
 		)
-		(property "Footprint" ""
+		(property "Footprint" "Package_DIP:DIP-8_W7.62mm_LongPads"
 			(at 26.67 138.43 0)
 			(effects
@@
 			)
 		)
-		(property "Footprint" ""
+		(property "Footprint" "Package_DIP:DIP-8_W7.62mm_LongPads"
 			(at 90.17 46.99 0)
 			(effects
@@
 	(symbol
 		(lib_id "Device:R")
-		(at 46.99 63.5 90)
+		(at 52.07 63.5 90)
 		(unit 1)
 		(exclude_from_sim no)
@@
 		(fields_autoplaced yes)
 		(property "Reference" "R3"
-			(at 46.99 57.15 90)
+			(at 52.07 57.15 90)
 			(effects
 				(font
@@
 			)
 		)
-		(property "Value" "2M"
-			(at 46.99 59.69 90)
+		(property "Value" "1М"
+			(at 52.07 59.69 90)
 			(effects
 				(font
@@
 		)
 		(property "Footprint" "Resistor_THT:R_Axial_DIN0204_L3.6mm_D1.6mm_P7.62mm_Horizontal"
-			(at 46.99 65.278 90)
+			(at 52.07 65.278 90)
 			(effects
 				(font
@@
 		)
 		(property "Datasheet" "~"
-			(at 46.99 63.5 0)
+			(at 52.07 63.5 0)
 			(effects
 				(font
@@
 		)
 		(property "Description" "Resistor"
-			(at 46.99 63.5 0)
+			(at 52.07 63.5 0)
 			(effects
 				(font
